File: 50 pin ribbon adapter/50 pin ribbon adapter.kicad_pcb (KiCad board)
At the start: 2 copper layers, 14 x 64.8 mm, 4 parts, among them J1 Conn_01x25_Socket, J2 Conn_01x25_Socket, J3 Conn_02x25_Odd_Even

Commit message: fixed silk
Other:
- board text added: "Adapter for 0.2{dblquote} spacing card edge connector pins to standard 50 pin ribbon"
- board text removed: "Adapter for 0.3{dblquote} spacing card edge connector pins to standard 50 pin ribbon"
Changed lines of the file:
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@@
   (gr_rect (start 140.335 36.195) (end 154.305 100.965)
     (stroke (width 0.1) (type default)) (fill none) (layer "Edge.Cuts"))
-  (gr_text "Adapter for 0.3{dblquote} spacing card edge connector pins to standard 50 pin ribbon" (at 150.495 37.465 90) (layer "B.SilkS")
+  (gr_text "Adapter for 0.2{dblquote} spacing card edge connector pins to standard 50 pin ribbon" (at 150.495 37.465 90) (layer "B.SilkS")
     (effects (font (size 1 1) (thickness 0.15)) (justify left bottom mirror))
   )
